File: PCB/otto_single_sided.brd (EAGLE design)
At the start: 57.2 x 53.3 mm, 19 parts, among them M1 ARDUINO-NANO-3.0, M2 SMALL_SERVO, M3 SMALL_SERVO, M4 SMALL_SERVO, M5 SMALL_SERVO

Commit message: connected R1 GND Point
R1 was not connected to GND
Connections:
- net GND: now also R1.2
Routing:
- net GND: track 240.5 -> 243.0 mm
Changed lines of the file:
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@@
 <wire x1="21.238" y1="15.484" x2="24" y2="14.5" width="0.6" layer="16"/>
 <wire x1="21.238" y1="18.746" x2="21.238" y2="15.484" width="0.6" layer="16"/>
+<contactref element="R1" pad="2"/>
+<wire x1="34.29" y1="29.21" x2="34.29" y2="31.75" width="0.6096" layer="16"/>
 </signal>
 <signal name="+5V">
